Commit message: Fix RGBD depth clip shadowing
gazebo_rgbd redefined min_depth/max_depth as properties, so callers' values were ignored and every RGBD camera clipped at 0.52-6.0 m.

File: gz_camera_macros/urdf/rgbd_camera.gazebo.xacro (robot description, xacro)
@@ -33,6 +33,4 @@
     <xacro:property name="cx" value="${image_width * 0.5}" />
     <xacro:property name="cy" value="${image_height * 0.5}" />
-    <xacro:property name="min_depth" value="0.52" />
-    <xacro:property name="max_depth" value="6.0" />
     <gazebo reference="${name}_color_frame">
         <sensor name="${name}" type="rgbd_camera">
